File: eagle/diagnostic_tool.brd (EAGLE design)
At the start: 160 x 100 mm, 9 parts, among them T1 PT204-6C

Commit message: Fixed buffer amp.
Connections:
- new net N$5: R1.1, SENSOR1.1, U$1.3
- net N$3: no longer R1.1, SENSOR1.1, U$1.3
Changed lines of the file:
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@@
 <contactref element="U$1" pad="1"/>
 <contactref element="LED1" pad="C@1"/>
+<contactref element="SG1" pad="1"/>
 <contactref element="U$1" pad="4"/>
-<contactref element="U$1" pad="3"/>
-<contactref element="R1" pad="1"/>
-<contactref element="SENSOR1" pad="1"/>
-<contactref element="SG1" pad="1"/>
-<wire x1="58.1" y1="39.34" x2="58.1" y2="41.94" width="0" layer="19" extent="1-1"/>
-<wire x1="56.2" y1="39.34" x2="58.1" y2="39.34" width="0" layer="19" extent="1-1"/>
-<wire x1="1.27" y1="-10.16" x2="56.2" y2="39.34" width="0" layer="19" extent="1-1"/>
-<wire x1="-2.54" y1="-13.47" x2="1.27" y2="-10.16" width="0" layer="19" extent="1-1"/>
-<wire x1="-2.54" y1="-26.67" x2="-2.54" y2="-13.47" width="0" layer="19" extent="1-1"/>
-<wire x1="-16.4592" y1="-29.845" x2="-2.54" y2="-26.67" width="0" layer="19" extent="1-1"/>
+<wire x1="56.2" y1="39.34" x2="58.1" y2="41.94" width="0" layer="19" extent="1-1"/>
+<wire x1="-2.54" y1="-13.47" x2="56.2" y2="39.34" width="0" layer="19" extent="1-1"/>
+<wire x1="-16.4592" y1="-29.845" x2="-2.54" y2="-13.47" width="0" layer="19" extent="1-1"/>
 </signal>
 <signal name="N$1">
@@
 <contactref element="T1" pad="E"/>
 </signal>
+<signal name="N$5">
+<contactref element="U$1" pad="3"/>
+<contactref element="R1" pad="1"/>
+<contactref element="SENSOR1" pad="1"/>
+<wire x1="1.27" y1="-10.16" x2="58.1" y2="39.34" width="0" layer="19" extent="1-1"/>
+<wire x1="-2.54" y1="-26.67" x2="1.27" y2="-10.16" width="0" layer="19" extent="1-1"/>
+</signal>
 </signals>
